Commit message: navigation is added

File: src/gazebo_sim/urdf/prototype.gazebo.xacro (robot description, xacro)
@@ -15,5 +15,5 @@
     <gravity> 1 </gravity>
     <mu1>100</mu1>
-    <mu2>100</mu2>-->
+    <mu2>100</mu2>
     <material>Gazebo/Black</material>
   </gazebo>
@@ -28,5 +28,5 @@
     <gravity> 1 </gravity>
     <mu1>100</mu1>
-    <mu2>100</mu2>-->
+    <mu2>100</mu2>
     <material>Gazebo/Black</material>
     <!--<material>Gazebo/Green</material>-->
@@ -43,5 +43,5 @@
     <gravity> 1 </gravity>
     <mu1>100</mu1>
-    <mu2>100</mu2>-->
+    <mu2>100</mu2>
     <material>Gazebo/Black</material>
     <!--<material>Gazebo/Green</material>-->
@@ -95,5 +95,5 @@
      <always_on>true</always_on>
      <visualize>true</visualize>
-     <update_rate>100</update_rate>
+     <update_rate>10</update_rate>
      <plugin name="laser_controller" filename="libgazebo_ros_ray_sensor.so">
       <ros>
@@ -111,5 +111,5 @@
         <remapping>~/out:=joint_states</remapping>
       </ros>
-      <update_rate>30</update_rate>
+      <update_rate>100</update_rate>
       <joint_name>front_left_wheel_joint</joint_name>
       <joint_name>front_right_wheel_joint</joint_name>
@@ -122,4 +122,5 @@
   <gazebo>
     <plugin filename="libgazebo_ros_diff_drive.so" name="prototype_diff_drive">
+      <update_rate>500</update_rate>
       <num_wheel_pairs>2</num_wheel_pairs>
       <!-- wheels -->

File: src/prototype/urdf/Battery_Control.xacro (robot description, xacro)
@@ -7,8 +7,8 @@
 <xacro:box_link name="Battery" mass="2.255" ixx="0.37583333" iyy="0.8333333"
 izz="0.8333333" box="0.15 0.060 0.095"/>
-<xacro:fixed_joint name="Battery_joint" origin="0.0 0.0 0.052" parent="base_link" child="Battery"/>
+<xacro:fixed_joint name="Battery_joint" origin="0.0 0.0 0.052" parent="chassis" child="Battery"/>
 <xacro:box_link name="control_board" mass="0.500" ixx="0.8333333" iyy="0.8333333"
 izz="0.37583333" box="0.15 0.060 0.095"/>
 <xacro:fixed_joint name="control_board_joint" origin="0.0 0.081 0.052"
-parent="base_link" child="control_board" />
+parent="chassis" child="control_board" />
 </robot>

File: src/prototype/urdf/crane.xacro (robot description, xacro)
@@ -7,5 +7,5 @@
 izz="0.4166667" box="0.06 0.2 0.06" FilePath="package://prototype/meshes/crane.dae"
 collision="0.0 -0.1 0.0"/>
-<xacro:fixed_joint name="crane_joint" origin="0.0 -0.12 0.032" parent="base_link"
+<xacro:fixed_joint name="crane_joint" origin="0.0 -0.12 0.032" parent="chassis"
 child="crane"/>
 <!-- ======================shaft_link & shaft_joint=======================-->
@@ -13,5 +13,5 @@
 <joint name="shaft_joint" type="continuous">
     <origin rpy="0.0 0.0 0.0" xyz="0 -0.44 0.0425" />
-    <parent link="base_link"/>
+    <parent link="chassis"/>
     <child link="shaft"/>
     <axis xyz="0.0 0.0 1.0"/>

File: src/prototype/urdf/lidar.xacro (robot description, xacro)
@@ -26,5 +26,5 @@
     <child link="laser_scan_frame"/>
     <axis xyz="0.0 0.0 0.0"/>-->
-    <parent link="base_link"/>
+    <parent link="chassis"/>
     <child link="laser_scan_frame"/>
     <axis xyz="0 0 1"/>

File: src/prototype/urdf/prototype.xacro (robot description, xacro)
@@ -9,5 +9,5 @@
 <!--<xacro:include filename="$(find prototype)/urdf/Battery_Control.xacro"/>-->
 <!--<xacro:include filename="$(find prototype)/urdf/crane.xacro"/>-->
-<xacro:include filename="$(find prototype)/urdf/hardware_interface.xacro"/>
+<!--<xacro:include filename="$(find prototype)/urdf/hardware_interface.xacro"/>-->
 <!--=========================xacro:properties=============================-->
     <xacro:property name="body_length" value="0.3"/>
@@ -17,20 +17,22 @@
 <!--***********************************************************************-->
   <!--=====================Base-Footprint and base_link link=================-->
-  <link name="base_footprint"/>
-  <!--<joint name="base_link_1_joint" type="fixed">
-    <parent link="base_footprint"/>
-    <child link="base_link_1"/>
-    <origin xyz="0.0 0.0 0.0" rpy="0.0 0.0 0.0"/>
-  </joint>
-  <xacro:box_link name="base_link_1" mass="1.21" ixx="0.0010803" iyy="0.00010259"
-  izz="0.00129793" box="0.1 0.1 0.2"/>-->
- <joint name="base_link_joint" type="fixed">
-  <origin rpy="0 0 0" xyz="0 0 0"/>
-  <parent link="base_footprint"/>
-  <child link="base_link"/>
+  <!-- BASE LINK-->
+  <link name="base_link">
+  </link>
+  <joint name="base_footprint_joint" type="fixed">
+    <parent link="base_link"/>
+    <child link="base_footprint"/>
+    <origin xyz="0 0 0" rpy="0 0 0"/>
+</joint>
+<link name="base_footprint">
+</link>
+ <joint name="chassis_joint" type="fixed">
+  <origin rpy="0 0 1.57" xyz="0 0 0"/>
+  <parent link="base_link"/>
+  <child link="chassis"/>
   <axis xyz="0 0 0"/>
   <joint_proprties damping ="0.0" friction="0.1"/>
  </joint>
- <xacro:box_link_meshes name="base_link" mass="1.21" ixx="0.0010803" iyy="0.00010259"
+ <xacro:box_link_meshes name="chassis" mass="1.21" ixx="0.0010803" iyy="0.00010259"
  izz="0.00129793" box="0.155 0.3 0.01" FilePath="package://prototype/meshes/blender_mesh.stl"
  collision="0.0 -0.1 0.0"/>

File: src/prototype/urdf/wheel.xacro (robot description, xacro)
@@ -31,14 +31,14 @@
    <!-- *********************wheel links and joints***************************************-->
  <xacro:joint name="front_right_wheel_joint" origin="-0.0900 -0.12 -0.025"
- parent="base_link" child="front_right_wheel"/>
+ parent="chassis" child="front_right_wheel"/>
 <xacro:wheel wheel_name="front_right_wheel"/>
 <xacro:joint name="front_left_wheel_joint" origin="0.0900 -.12 -0.025"
-parent="base_link" child="front_left_wheel" />
+parent="chassis" child="front_left_wheel" />
 <xacro:wheel wheel_name="front_left_wheel"/>
 <xacro:joint name="back_right_wheel_joint" origin="-0.0900 0.12 -0.025"
-parent="base_link" child="back_right_wheel"/>
+parent="chassis" child="back_right_wheel"/>
 <xacro:wheel  wheel_name="back_right_wheel"/>
 <xacro:joint name="back_left_wheel_joint" origin="0.0900 0.12 -0.025"
-parent="base_link" child="back_left_wheel"/>
+parent="chassis" child="back_left_wheel"/>
 <xacro:wheel  wheel_name="back_left_wheel"/>
 </robot>
