Commit message: updated robotlocal

File: src/prototype/urdf/camera.xacro (robot description, xacro)
@@ -4,12 +4,15 @@
 <link name="camera_link">
     <visual>
-        <origin xyz="0 0 0" rpy="0.0 0.0 0.0"/>
+        <origin xyz="0 0 0.0" rpy="0.0 0.0 0.0"/>
         <geometry>
         <box size="0.010 0.03 0.03"/>
         </geometry>
+        <material name="black">
+          <color rgba="0.0 0.0 0.0 1.0"/>
+        </material>
        </visual>
 </link>
 <joint name="camera_joint" type="fixed">
-    <origin xyz="0.0900 0.0 0.15" rpy="0.0 0.0 0.0"/>
+    <origin xyz="0.15 0.0 0.05" rpy="0.0 0.0 0.0"/>
     <parent link="chassis"/>
     <child link="camera_link"/>
@@ -18,7 +21,18 @@
     <origin xyz="0.0 0.0 0.0" rpy="-1.57 0.0 -1.57"/>
     <parent link="camera_link"/>
+     <!--<axis xyz="1.0 1.0 1.0"/>-->
     <child link="camera_link_optical"/>
 </joint>
 <link name="camera_link_optical">
 </link>
+<!--
+<joint name="object_joint" type="continuous">
+    <origin xyz="0.0 0.0 0.0" rpy="0.0 0.0 0.0"/>
+    <parent link="camera_link_optical"/>
+     <axis xyz="1.0 1.0 1.0"/>
+    <child link="object_link"/>
+</joint>
+<link name="object_link">
+</link>
+-->
 </robot>

File: src/prototype/urdf/joint_macros.xacro (robot description, xacro)
@@ -4,10 +4,10 @@
     <xacro:property name="wheel_length" value="0.026"/>
    <!--===============xacro for continuous joints=========================-->
-    <xacro:macro name="joint" params="name origin parent child">
-        <joint name="${name}" type="continuous">
+    <xacro:macro name="joint_wheel" params="name origin parent child">
+        <joint name="${name}" type="fixed">
             <origin xyz="${origin}" rpy="0.0 0.0 0.0"/>
             <parent link="${parent}"/>
             <child link="${child}"/>
-            <axis xyz="1 0.0 0.0"/>
+            <axis xyz="0.0 1.0 0.0"/>
             <limit effort="200" velocity="2.0"/>
             <joint_properties damping="1.1" friction="1.0"/>

File: src/prototype/urdf/prototype.xacro (robot description, xacro)
@@ -6,6 +6,4 @@
 <xacro:include filename="$(find prototype)/urdf/joint_macros.xacro"/>
 <xacro:include filename="$(find prototype)/urdf/link_macros.xacro"/>
-<xacro:include filename="$(find prototype)/urdf/Battery_Control.xacro"/>
-<xacro:include filename="$(find prototype)/urdf/crane.xacro"/>
 <xacro:include filename="$(find prototype)/urdf/hardware_interface.xacro"/>
 <xacro:include filename="$(find prototype)/urdf/camera.xacro"/>
@@ -28,5 +26,5 @@
 </link>
  <joint name="chassis_joint" type="fixed">
-  <origin rpy="0 0 1.57" xyz="0 0 0"/>
+  <origin rpy="0 0 0.0" xyz="0 0 0.062"/>
   <parent link="base_link"/>
   <child link="chassis"/>
@@ -34,21 +32,17 @@
   <joint_proprties damping ="0.0" friction="0.1"/>
  </joint>
- <xacro:box_link_meshes name="chassis" mass="1.21" ixx="0.0010803" iyy="0.00010259"
- izz="0.00129793" box="0.155 0.3 0.01" FilePath="package://prototype/meshes/blender_mesh.stl"
- collision="0.0 -0.1 0.0"/>
-<!--
- <xacro:box_link name="base_link" mass="1.21" ixx="0.0010803" iyy="0.00010259"
- izz="0.00129793" box="0.155 0.3 0.01"/>-->
- <joint name="imu_joint" type="fixed">
-  <parent link="chassis"/>
-  <child link="imu_link"/>
-  <origin xyz="0.0 0.0 0.0" rpy="0.0 0.0 0.0"/>
- </joint>
- <link name="imu_link"></link>
+<link name="chassis">
+    <visual>
+        <origin xyz="0 0 0.075" rpy="0.0 0.0 0.0"/>
+        <geometry>
+        <box size="0.3 0.155 0.15"/>
+        </geometry>
+       </visual>
+</link>
  <joint name="caster_wheel_joint" type="fixed">
   <parent link="chassis"/>
   <child link="caster_wheel"/>
   <axis xyz="0 0 0"/>
-  <origin xyz="0.0 -0.10 -0.020" rpy="0 0 0"/>
+  <origin xyz="0.125 0.0 -0.038" rpy="0 0 0"/>
  </joint>
         <link name="caster_wheel">
@@ -56,5 +50,5 @@
                 <origin xyz="0.0 0.0 0.0" rpy="0.0 0.0 0.0"/>
                 <geometry>
-                 <sphere radius="0.021"/>
+                 <sphere radius="0.025"/>
                 </geometry>
                 <material name="blue">
@@ -62,16 +56,4 @@
                 </material>
             </visual>
-            <collision>
-                <origin xyz="0.0 0.0 0.0" rpy="0.0 1.5707 0.0"/>
-                <geometry>
-                    <sphere radius="0.021"/>/>
-                </geometry>
-            </collision>
-            <inertial>
-                <origin rpy="0 0 0" xyz="0 0 0"/>
-                <mass value="0.034"/>
-              <inertia ixx="1.37e-5" ixy="0" ixz="0" iyy="1.37e-5" iyz="0" izz="3.41e-6"/>
-              </inertial>
-              <dynamics damping="0.5" friction="0.1"/>
  </link>
 </robot>

Commit message: updated the sensors and localization

File: src/prototype/urdf/camera.xacro (robot description, xacro)
@@ -4,12 +4,15 @@
 <link name="camera_link">
     <visual>
-        <origin xyz="0 0 0" rpy="0.0 0.0 0.0"/>
+        <origin xyz="0 0 0.0" rpy="0.0 0.0 0.0"/>
         <geometry>
         <box size="0.010 0.03 0.03"/>
         </geometry>
+        <material name="black">
+          <color rgba="0.0 0.0 0.0 1.0"/>
+        </material>
        </visual>
 </link>
 <joint name="camera_joint" type="fixed">
-    <origin xyz="0.0900 0.0 0.15" rpy="0.0 0.0 0.0"/>
+    <origin xyz="0.15 0.0 0.05" rpy="0.0 0.0 0.0"/>
     <parent link="chassis"/>
     <child link="camera_link"/>

File: src/prototype/urdf/hardware_interface.xacro (robot description, xacro)
@@ -12,5 +12,5 @@
           <param name="back_right_wheel_name">back_right_wheel_joint</param>
           <param name="loop_rate">30</param>
-          <param name="device">/dev/serial/by-path/platform-xhci-hcd.3.auto-usb-0:1:1.0</param>
+          <param name="device">/dev/serial/by-path/platform-fd500000.pcie-pci-0000:01:00.0-usb-0:1.4:1.0</param>
           <param name="baud_rate">115200</param>
           <param name="timeout">1000</param>

File: src/prototype/urdf/joint_macros.xacro (robot description, xacro)
@@ -4,10 +4,10 @@
     <xacro:property name="wheel_length" value="0.026"/>
    <!--===============xacro for continuous joints=========================-->
-    <xacro:macro name="joint" params="name origin parent child">
+    <xacro:macro name="joint_wheel" params="name origin parent child">
         <joint name="${name}" type="continuous">
             <origin xyz="${origin}" rpy="0.0 0.0 0.0"/>
             <parent link="${parent}"/>
             <child link="${child}"/>
-            <axis xyz="1 0.0 0.0"/>
+            <axis xyz="0.0 1.0 0.0"/>
             <limit effort="200" velocity="2.0"/>
             <joint_properties damping="1.1" friction="1.0"/>

File: src/prototype/urdf/lidar.xacro (robot description, xacro)
@@ -22,8 +22,5 @@
 </link>
 <joint name="laser_scan_frame_joint" type="fixed">
-    <origin xyz="0.0 0.0 0.15" rpy="0.0 0.0 -1.57"/>
-    <!--<parent link="laser_scan_link"/>
-    <child link="laser_scan_frame"/>
-    <axis xyz="0.0 0.0 0.0"/>-->
+    <origin xyz="0.0 0.0 0.248" rpy="0.0 0.0 0.0"/>
     <parent link="chassis"/>
     <child link="laser_scan_frame"/>

File: src/prototype/urdf/link_macros.xacro (robot description, xacro)
@@ -5,23 +5,13 @@
   <xacro:macro name="box_link" params="name mass ixx iyy izz box">
     <link name="${name}">
-     <inertial>
-        <origin xyz="0.0 0.0 0.0" rpy="0.0 0.0 0.0"/>
-        <mass value="${mass}"/>
-        <inertia ixx="${ixx}" ixy="0.0" ixz="0.0" iyy="${iyy}" iyz="0.0" izz="${izz}"/>
-     </inertial>
      <visual>
+     <origin xyz="0 0 0" rpy="0 0 0"/>
         <geometry>
             <box size="${box}"/>
         </geometry>
-        <material name="">
+        <material name="red">
             <color rgba="1.0 0.0 0.0 1.0"/>
         </material>
      </visual>
-     <collision>
-        <origin xyz="0.0 0.0 0.0" rpy="0.0 0.0 0.0"/>
-        <geometry>
-            <box size="${box}"/>
-        </geometry>
-     </collision>
      </link>
  </xacro:macro>

File: src/prototype/urdf/prototype.xacro (robot description, xacro)
@@ -6,9 +6,6 @@
 <xacro:include filename="$(find prototype)/urdf/joint_macros.xacro"/>
 <xacro:include filename="$(find prototype)/urdf/link_macros.xacro"/>
-<xacro:include filename="$(find prototype)/urdf/Battery_Control.xacro"/>
-<xacro:include filename="$(find prototype)/urdf/crane.xacro"/>
 <xacro:include filename="$(find prototype)/urdf/hardware_interface.xacro"/>
 <xacro:include filename="$(find prototype)/urdf/camera.xacro"/>
-<xacro:include filename="$(find prototype)/urdf/pillar.xacro"/>
 <!--=========================xacro:properties=============================-->
     <xacro:property name="body_length" value="0.3"/>
@@ -29,5 +26,5 @@
 </link>
  <joint name="chassis_joint" type="fixed">
-  <origin rpy="0 0 1.57" xyz="0 0 0"/>
+  <origin rpy="0 0 0.0" xyz="0 0 0.062"/>
   <parent link="base_link"/>
   <child link="chassis"/>
@@ -35,27 +32,23 @@
   <joint_proprties damping ="0.0" friction="0.1"/>
  </joint>
- <xacro:box_link_meshes name="chassis" mass="1.21" ixx="0.0010803" iyy="0.00010259"
- izz="0.00129793" box="0.155 0.3 0.01" FilePath="package://prototype/meshes/blender_mesh.stl"
- collision="0.0 -0.1 0.0"/>
-<!--
- <xacro:box_link name="base_link" mass="1.21" ixx="0.0010803" iyy="0.00010259"
- izz="0.00129793" box="0.155 0.3 0.01"/>-->
- <joint name="imu_joint" type="fixed">
-  <parent link="chassis"/>
-  <child link="imu_link"/>
-  <origin xyz="0.0 0.0 0.0" rpy="0.0 0.0 0.0"/>
- </joint>
- <link name="imu_link"></link>
+<link name="chassis">
+    <visual>
+        <origin xyz="0 0 0.075" rpy="0.0 0.0 0.0"/>
+        <geometry>
+        <box size="0.3 0.155 0.15"/>
+        </geometry>
+       </visual>
+</link>
  <joint name="caster_wheel_joint" type="fixed">
   <parent link="chassis"/>
   <child link="caster_wheel"/>
   <axis xyz="0 0 0"/>
-  <origin xyz="0.0 -0.10 -0.020" rpy="0 0 0"/>
+  <origin xyz="0.125 0.0 -0.038" rpy="0 0 0"/>
  </joint>
-        <link name="caster_wheel">
+ <link name="caster_wheel">
             <visual>
                 <origin xyz="0.0 0.0 0.0" rpy="0.0 0.0 0.0"/>
                 <geometry>
-                 <sphere radius="0.021"/>
+                 <sphere radius="0.025"/>
                 </geometry>
                 <material name="blue">
@@ -63,16 +56,11 @@
                 </material>
             </visual>
-            <collision>
-                <origin xyz="0.0 0.0 0.0" rpy="0.0 1.5707 0.0"/>
-                <geometry>
-                    <sphere radius="0.021"/>/>
-                </geometry>
-            </collision>
-            <inertial>
-                <origin rpy="0 0 0" xyz="0 0 0"/>
-                <mass value="0.034"/>
-              <inertia ixx="1.37e-5" ixy="0" ixz="0" iyy="1.37e-5" iyz="0" izz="3.41e-6"/>
-              </inertial>
-              <dynamics damping="0.5" friction="0.1"/>
  </link>
+ <joint name="imu_joint" type="fixed">
+  <parent link="chassis"/>
+  <child link="imu_link"/>
+  <axis xyz="0.0 0.0 1.0"/>
+  <origin xyz="0.0 0.0 1.00" rpy="0.0 0.0 0.0"/>
+ </joint>
+ <link name="imu_link"></link>
 </robot>

File: src/prototype/urdf/wheel.xacro (robot description, xacro)
@@ -7,5 +7,5 @@
         <link name="${wheel_name}">
             <visual>
-                <origin xyz="0.0 0.0 0.0" rpy="0.0 1.5707 0.0"/>
+                <origin xyz="0.0 0.0 0.0" rpy="1.57 0.0 0.0"/>
                 <geometry>
                  <cylinder radius="${wheel_radius}" length="${wheel_length}"/>
@@ -30,8 +30,8 @@
    </xacro:macro>
    <!-- *********************wheel links and joints***************************************-->
-<xacro:joint name="back_right_wheel_joint" origin="-0.0900 0.12 -0.025"
+<xacro:joint_wheel name="back_right_wheel_joint" origin="-0.0900 -0.088 -0.025"
 parent="chassis" child="back_right_wheel"/>
 <xacro:wheel  wheel_name="back_right_wheel"/>
-<xacro:joint name="back_left_wheel_joint" origin="0.0900 0.12 -0.025"
+<xacro:joint_wheel name="back_left_wheel_joint" origin="-0.0900 0.088 -0.025"
 parent="chassis" child="back_left_wheel"/>
 <xacro:wheel  wheel_name="back_left_wheel"/>

Commit message: updated the nav2 config

File: src/prototype/urdf/camera.xacro (robot description, xacro)
@@ -15,5 +15,5 @@
 <joint name="camera_joint" type="fixed">
     <origin xyz="0.15 0.0 0.05" rpy="0.0 0.0 0.0"/>
-    <parent link="chassis"/>
+    <parent link="base_link"/>
     <child link="camera_link"/>
 </joint>

File: src/prototype/urdf/hardware_interface.xacro (robot description, xacro)
@@ -12,5 +12,5 @@
           <param name="back_right_wheel_name">back_right_wheel_joint</param>
           <param name="loop_rate">30</param>
-          <param name="device">/dev/serial/by-path/platform-fd500000.pcie-pci-0000:01:00.0-usb-0:1.4:1.0</param>
+          <param name="device">/dev/serial/by-path/platform-fd500000.pcie-pci-0000:01:00.0-usb-0:1.1:1.0</param>
           <param name="baud_rate">115200</param>
           <param name="timeout">1000</param>

File: src/prototype/urdf/lidar.xacro (robot description, xacro)
@@ -2,5 +2,5 @@
 <!--=========================starting xacros================================-->
 <robot xmlns:xacro="http://www.ros.org/wiki/xacro" name="prototype">
-<link name="laser_scan_frame">
+<link name="base_laser">
     <visual>
         <origin xyz="0 0 0" rpy="0.0 0.0 0.0"/>
@@ -21,8 +21,8 @@
          </inertial>
 </link>
-<joint name="laser_scan_frame_joint" type="fixed">
+<joint name="base_laser_joint" type="fixed">
     <origin xyz="0.0 0.0 0.248" rpy="0.0 0.0 0.0"/>
-    <parent link="chassis"/>
-    <child link="laser_scan_frame"/>
+    <parent link="base_link"/>
+    <child link="base_laser"/>
     <axis xyz="0 0 1"/>
     <limit lower="-0.1" upper="0.0" effort="20.0" velocity="2.0"/>

File: src/prototype/urdf/prototype.xacro (robot description, xacro)
@@ -17,29 +17,19 @@
   <!-- BASE LINK-->
   <link name="base_link">
-  </link>
-  <joint name="base_footprint_joint" type="fixed">
-    <parent link="base_link"/>
-    <child link="base_footprint"/>
-    <origin xyz="0 0 0" rpy="0 0 0"/>
-</joint>
-<link name="base_footprint">
-</link>
- <joint name="chassis_joint" type="fixed">
-  <origin rpy="0 0 0.0" xyz="0 0 0.062"/>
-  <parent link="base_link"/>
-  <child link="chassis"/>
-  <axis xyz="0 0 0"/>
-  <joint_proprties damping ="0.0" friction="0.1"/>
- </joint>
-<link name="chassis">
-    <visual>
-        <origin xyz="0 0 0.075" rpy="0.0 0.0 0.0"/>
+   <visual>
         <geometry>
         <box size="0.3 0.155 0.15"/>
         </geometry>
        </visual>
+  </link>
+  <joint name="base_joint" type="fixed">
+    <parent link="base_link"/>
+    <child link="base_footprint"/>
+    <origin xyz="0 0 -0.091" rpy="0 0 0"/>
+</joint>
+<link name="base_footprint">
 </link>
  <joint name="caster_wheel_joint" type="fixed">
-  <parent link="chassis"/>
+  <parent link="base_link"/>
   <child link="caster_wheel"/>
   <axis xyz="0 0 0"/>
@@ -58,5 +48,5 @@
  </link>
  <joint name="imu_joint" type="fixed">
-  <parent link="chassis"/>
+  <parent link="base_link"/>
   <child link="imu_link"/>
   <axis xyz="0.0 0.0 1.0"/>

File: src/prototype/urdf/wheel.xacro (robot description, xacro)
@@ -30,9 +30,9 @@
    </xacro:macro>
    <!-- *********************wheel links and joints***************************************-->
-<xacro:joint_wheel name="back_right_wheel_joint" origin="-0.0900 -0.088 -0.025"
-parent="chassis" child="back_right_wheel"/>
+<xacro:joint_wheel name="back_right_wheel_joint" origin="-0.0900 -0.088 -0.075"
+parent="base_link" child="back_right_wheel"/>
 <xacro:wheel  wheel_name="back_right_wheel"/>
-<xacro:joint_wheel name="back_left_wheel_joint" origin="-0.0900 0.088 -0.025"
-parent="chassis" child="back_left_wheel"/>
+<xacro:joint_wheel name="back_left_wheel_joint" origin="-0.0900 0.088 -0.075"
+parent="base_link" child="back_left_wheel"/>
 <xacro:wheel  wheel_name="back_left_wheel"/>
 </robot>

Commit message: updated the urdf

File: src/prototype/urdf/camera.xacro (robot description, xacro)
@@ -15,5 +15,5 @@
 <joint name="camera_joint" type="fixed">
     <origin xyz="0.15 0.0 0.05" rpy="0.0 0.0 0.0"/>
-    <parent link="base_link"/>
+    <parent link="chassis"/>
     <child link="camera_link"/>
 </joint>

File: src/prototype/urdf/joint_macros.xacro (robot description, xacro)
@@ -1,5 +1,5 @@
 <?xml version="1.0"?>
 <robot xmlns:xacro="http://www.ros.org/wiki/xacro" name="prototype">
-    <xacro:property name="wheel_radius" value="0.032"/>
+    <xacro:property name="wheel_radius" value="0.05"/>
     <xacro:property name="wheel_length" value="0.026"/>
    <!--===============xacro for continuous joints=========================-->

File: src/prototype/urdf/lidar.xacro (robot description, xacro)
@@ -22,6 +22,6 @@
 </link>
 <joint name="base_laser_joint" type="fixed">
-    <origin xyz="0.0 0.0 0.248" rpy="0.0 0.0 0.0"/>
-    <parent link="base_link"/>
+    <origin xyz="0.0 0.0 0.222" rpy="0.0 0.0 0.0"/>
+    <parent link="chassis"/>
     <child link="base_laser"/>
     <axis xyz="0 0 1"/>

File: src/prototype/urdf/link_macros.xacro (robot description, xacro)
@@ -6,5 +6,5 @@
     <link name="${name}">
      <visual>
-     <origin xyz="0 0 0" rpy="0 0 0"/>
+     <origin xyz="0 0 0.1" rpy="0 0 0"/>
         <geometry>
             <box size="${box}"/>

File: src/prototype/urdf/prototype.xacro (robot description, xacro)
@@ -9,30 +9,39 @@
 <xacro:include filename="$(find prototype)/urdf/camera.xacro"/>
 <!--=========================xacro:properties=============================-->
-    <xacro:property name="body_length" value="0.3"/>
-    <xacro:property name="body_width" value="0.155"/>
-    <xacro:property name="body_height" value="0.01"/>
+    <xacro:property name="body_length" value="0.41"/>
+    <xacro:property name="body_width" value="0.41"/>
+    <xacro:property name="body_height" value="0.82"/>
                               <!-- end of xacros-->
 <!--***********************************************************************-->
   <!--=====================Base-Footprint and base_link link=================-->
   <!-- BASE LINK-->
-  <link name="base_link">
-   <visual>
-        <geometry>
-        <box size="0.3 0.155 0.15"/>
-        </geometry>
-       </visual>
-  </link>
+  <link name="base_link"></link>
   <joint name="base_joint" type="fixed">
     <parent link="base_link"/>
     <child link="base_footprint"/>
-    <origin xyz="0 0 -0.091" rpy="0 0 0"/>
-</joint>
+    <origin xyz="0.0 0.0 0.0" rpy="0 0 0"/>
+  </joint>
 <link name="base_footprint">
 </link>
+ <joint name="chassis_joint" type="fixed">
+    <parent link="base_link"/>
+    <child link="chassis"/>
+    <origin xyz="0.0 0.0 0.12" rpy="0 0 0"/>
+  </joint>
+<link name="chassis">
+    <visual>
+        <geometry>
+            <box size="0.4112 0.4112 0.04"/>
+        </geometry>
+        <material name="silver">
+            <color rgba="0.75 0.75 0.75 1.0"/> <!-- Silver color with RGBA values -->
+        </material>
+    </visual>
+</link>
  <joint name="caster_wheel_joint" type="fixed">
-  <parent link="base_link"/>
+  <parent link="chassis"/>
   <child link="caster_wheel"/>
   <axis xyz="0 0 0"/>
-  <origin xyz="0.125 0.0 -0.038" rpy="0 0 0"/>
+  <origin xyz="0.19 0.0 -0.10" rpy="0 0 0"/>
  </joint>
  <link name="caster_wheel">
@@ -42,11 +51,11 @@
                  <sphere radius="0.025"/>
                 </geometry>
-                <material name="blue">
-                    <color rgba="0.0 0.0 1.0 1.0"/>
+                <material name="white">
+                    <color rgba="1.0 1.0 1.0 1.0"/>
                 </material>
             </visual>
  </link>
  <joint name="imu_joint" type="fixed">
-  <parent link="base_link"/>
+  <parent link="chassis"/>
   <child link="imu_link"/>
   <axis xyz="0.0 0.0 1.0"/>

File: src/prototype/urdf/wheel.xacro (robot description, xacro)
@@ -11,6 +11,6 @@
                  <cylinder radius="${wheel_radius}" length="${wheel_length}"/>
                 </geometry>
-                <material name="blue">
-                    <color rgba="0.0 0.0 1.0 1.0"/>
+                <material name="black">
+                    <color rgba="0.0 0.0 0.0 1.0"/>
                 </material>
             </visual>
@@ -30,9 +30,9 @@
    </xacro:macro>
    <!-- *********************wheel links and joints***************************************-->
-<xacro:joint_wheel name="back_right_wheel_joint" origin="-0.0900 -0.088 -0.075"
-parent="base_link" child="back_right_wheel"/>
+<xacro:joint_wheel name="back_right_wheel_joint" origin="-0.1806 -0.225 -0.05"
+parent="chassis" child="back_right_wheel"/>
 <xacro:wheel  wheel_name="back_right_wheel"/>
-<xacro:joint_wheel name="back_left_wheel_joint" origin="-0.0900 0.088 -0.075"
-parent="base_link" child="back_left_wheel"/>
+<xacro:joint_wheel name="back_left_wheel_joint" origin="-0.1806 0.225 -0.05"
+parent="chassis" child="back_left_wheel"/>
 <xacro:wheel  wheel_name="back_left_wheel"/>
 </robot>
