Commit message: latest updates

File: src/prototype/urdf/camera.xacro (robot description, xacro)
@@ -14,5 +14,5 @@
 </link>
 <joint name="camera_joint" type="fixed">
-    <origin xyz="0.15 0.0 0.05" rpy="0.0 0.0 0.0"/>
+    <origin xyz="0.19 -0.20 0.675" rpy="3.14 0.0 0.0"/>
     <parent link="chassis"/>
     <child link="camera_link"/>
@@ -21,18 +21,7 @@
     <origin xyz="0.0 0.0 0.0" rpy="-1.57 0.0 -1.57"/>
     <parent link="camera_link"/>
-     <!--<axis xyz="1.0 1.0 1.0"/>-->
     <child link="camera_link_optical"/>
 </joint>
 <link name="camera_link_optical">
 </link>
-<!--
-<joint name="object_joint" type="continuous">
-    <origin xyz="0.0 0.0 0.0" rpy="0.0 0.0 0.0"/>
-    <parent link="camera_link_optical"/>
-     <axis xyz="1.0 1.0 1.0"/>
-    <child link="object_link"/>
-</joint>
-<link name="object_link">
-</link>
--->
 </robot>

File: src/prototype/urdf/hardware_interface.xacro (robot description, xacro)
@@ -12,5 +12,5 @@
           <param name="back_right_wheel_name">back_right_wheel_joint</param>
           <param name="loop_rate">30</param>
-          <param name="device">/dev/serial/by-path/platform-xhci-hcd.3.auto-usb-0:1:1.0</param>
+          <param name="device">/dev/serial/by-path/platform-fd500000.pcie-pci-0000:01:00.0-usb-0:1.1:1.0</param>
           <param name="baud_rate">115200</param>
           <param name="timeout">1000</param>

File: src/prototype/urdf/joint_macros.xacro (robot description, xacro)
@@ -1,9 +1,9 @@
 <?xml version="1.0"?>
 <robot xmlns:xacro="http://www.ros.org/wiki/xacro" name="prototype">
-    <xacro:property name="wheel_radius" value="0.032"/>
+    <xacro:property name="wheel_radius" value="0.05"/>
     <xacro:property name="wheel_length" value="0.026"/>
    <!--===============xacro for continuous joints=========================-->
     <xacro:macro name="joint_wheel" params="name origin parent child">
-        <joint name="${name}" type="fixed">
+        <joint name="${name}" type="continuous">
             <origin xyz="${origin}" rpy="0.0 0.0 0.0"/>
             <parent link="${parent}"/>

File: src/prototype/urdf/lidar.xacro (robot description, xacro)
@@ -2,5 +2,5 @@
 <!--=========================starting xacros================================-->
 <robot xmlns:xacro="http://www.ros.org/wiki/xacro" name="prototype">
-<link name="laser_scan_frame">
+<link name="base_laser">
     <visual>
         <origin xyz="0 0 0" rpy="0.0 0.0 0.0"/>
@@ -21,8 +21,8 @@
          </inertial>
 </link>
-<joint name="laser_scan_frame_joint" type="fixed">
-    <origin xyz="0.0 0.0 0.248" rpy="0.0 0.0 0.0"/>
+<joint name="base_laser_joint" type="fixed">
+    <origin xyz="0.0 0.0 0.222" rpy="0.0 0.0 0.0"/>
     <parent link="chassis"/>
-    <child link="laser_scan_frame"/>
+    <child link="base_laser"/>
     <axis xyz="0 0 1"/>
     <limit lower="-0.1" upper="0.0" effort="20.0" velocity="2.0"/>

File: src/prototype/urdf/prototype.xacro (robot description, xacro)
@@ -9,34 +9,33 @@
 <xacro:include filename="$(find prototype)/urdf/camera.xacro"/>
 <!--=========================xacro:properties=============================-->
-    <xacro:property name="body_length" value="0.3"/>
-    <xacro:property name="body_width" value="0.155"/>
-    <xacro:property name="body_height" value="0.01"/>
+    <xacro:property name="body_length" value="0.41"/>
+    <xacro:property name="body_width" value="0.41"/>
+    <xacro:property name="body_height" value="0.82"/>
                               <!-- end of xacros-->
 <!--***********************************************************************-->
   <!--=====================Base-Footprint and base_link link=================-->
   <!-- BASE LINK-->
-  <link name="base_link">
-  </link>
-  <joint name="base_footprint_joint" type="fixed">
+  <link name="base_link"></link>
+  <joint name="base_joint" type="fixed">
     <parent link="base_link"/>
     <child link="base_footprint"/>
     <origin xyz="0.0 0.0 0.0" rpy="0 0 0"/>
-</joint>
+  </joint>
 <link name="base_footprint">
 </link>
  <joint name="chassis_joint" type="fixed">
-  <origin rpy="0.0 0.0 0.0" xyz="0 0 0.062"/>
-  <parent link="base_link"/>
-  <child link="chassis"/>
-  <axis xyz="0 0 0"/>
-  <joint_proprties damping ="0.0" friction="0.1"/>
- </joint>
+    <parent link="base_link"/>
+    <child link="chassis"/>
+    <origin xyz="0.0 0.0 0.12" rpy="0 0 0"/>
+  </joint>
 <link name="chassis">
     <visual>
-        <origin xyz="0 0 0.075" rpy="0.0 0.0 0.0"/>
         <geometry>
-        <box size="0.3 0.155 0.15"/>
+            <box size="0.4112 0.4112 0.04"/>
         </geometry>
-       </visual>
+        <material name="silver">
+            <color rgba="0.75 0.75 0.75 1.0"/> <!-- Silver color with RGBA values -->
+        </material>
+    </visual>
 </link>
  <joint name="caster_wheel_joint" type="fixed">
@@ -44,7 +43,7 @@
   <child link="caster_wheel"/>
   <axis xyz="0 0 0"/>
-  <origin xyz="0.125 0.0 -0.038" rpy="0 0 0"/>
+  <origin xyz="0.19 0.0 -0.10" rpy="0 0 0"/>
  </joint>
-        <link name="caster_wheel">
+ <link name="caster_wheel">
             <visual>
                 <origin xyz="0.0 0.0 0.0" rpy="0.0 0.0 0.0"/>
@@ -52,8 +51,15 @@
                  <sphere radius="0.025"/>
                 </geometry>
-                <material name="blue">
-                    <color rgba="0.0 0.0 1.0 1.0"/>
+                <material name="white">
+                    <color rgba="1.0 1.0 1.0 1.0"/>
                 </material>
             </visual>
  </link>
+ <joint name="imu_joint" type="fixed">
+  <parent link="chassis"/>
+  <child link="imu_link"/>
+  <axis xyz="0.0 0.0 1.0"/>
+  <origin xyz="0.0 0.0 1.00" rpy="0.0 0.0 0.0"/>
+ </joint>
+ <link name="imu_link"></link>
 </robot>

File: src/prototype/urdf/wheel.xacro (robot description, xacro)
@@ -11,8 +11,7 @@
                  <cylinder radius="${wheel_radius}" length="${wheel_length}"/>
                 </geometry>
-                <material name="blue">
-                    <color rgba="0.0 0.0 1.0 1.0"/>
+                <material name="black">
+                    <color rgba="0.0 0.0 0.0 1.0"/>
                 </material>
-               /
             </visual>
             <collision>
@@ -31,8 +30,8 @@
    </xacro:macro>
    <!-- *********************wheel links and joints***************************************-->
-<xacro:joint_wheel name="back_right_wheel_joint" origin="-0.0900 -0.088 -0.025"
+<xacro:joint_wheel name="back_right_wheel_joint" origin="-0.1806 -0.225 -0.05"
 parent="chassis" child="back_right_wheel"/>
 <xacro:wheel  wheel_name="back_right_wheel"/>
-<xacro:joint_wheel name="back_left_wheel_joint" origin="-0.0900 0.088 -0.025"
+<xacro:joint_wheel name="back_left_wheel_joint" origin="-0.1806 0.225 -0.05"
 parent="chassis" child="back_left_wheel"/>
 <xacro:wheel  wheel_name="back_left_wheel"/>

Commit message: follow_me settings

File: src/prototype/urdf/camera.xacro (robot description, xacro)
@@ -14,5 +14,5 @@
 </link>
 <joint name="camera_joint" type="fixed">
-    <origin xyz="0.19 -0.20 0.675" rpy="3.14 0.0 0.0"/>
+    <origin xyz="0.19 -0.10 0.675" rpy="3.14 0.0 0.0"/>
     <parent link="chassis"/>
     <child link="camera_link"/>
