Commit message: updated motor_control and prototype

File: src/prototype/urdf/hardware_interface.xacro (robot description, xacro)
@@ -24,5 +24,5 @@
           <state_interface name="velocity" />
         </joint>
-        <joint name="front_right_wheel_joint">
+        <joint name="front_left_wheel_joint">
           <command_interface name="velocity">
             <param name="min">0.0</param>

Commit message: updating the prototype and motor_control

File: src/prototype/urdf/hardware_interface.xacro (robot description, xacro)
@@ -7,12 +7,15 @@
     <ros2_control name="PrototypeMotor" type="system">
         <hardware>
+          <!--<plugin>diffdrive_arduino/DiffDriveArduinoHardware</plugin>-->
           <plugin>motor_control/MotorControl</plugin>
-          <param name="left_wheel_name">front_left_wheel_joint</param>
-          <param name="right_wheel_name">front_right_wheel_joint</param>
+          <param name="front_left_wheel_name">front_left_wheel_joint</param>
+          <param name="front_right_wheel_name">front_right_wheel_joint</param>
+          <param name="back_left_wheel_name">back_left_wheel_joint</param>
+          <param name="back_right_wheel_name">back_right_wheel_joint</param>
           <param name="loop_rate">30</param>
           <param name="device">/dev/ttyACM0</param>
           <param name="baud_rate">115200</param>
-          <param name="timeout">5000</param>
-          <param name="enc_counts_per_rev">3436</param>
+          <param name="timeout">1000</param>
+          <param name="enc_counts_per_rev">120</param>
         </hardware>
         <joint name="front_right_wheel_joint">
@@ -32,4 +35,20 @@
           <state_interface name="velocity" />
         </joint>
+        <joint name="back_right_wheel_joint">
+          <command_interface name="velocity">
+            <param name="min">0.0</param>
+            <param name="max">2.0</param>
+          </command_interface>
+          <state_interface name="position" />
+          <state_interface name="velocity" />
+        </joint>
+        <joint name="back_left_wheel_joint">
+          <command_interface name="velocity">
+            <param name="min">0.0</param>
+            <param name="max">2.0</param>
+          </command_interface>
+          <state_interface name="position" />
+          <state_interface name="velocity" />
+        </joint>
       </ros2_control>
 </robot>

File: src/prototype/urdf/joint_macros.xacro (robot description, xacro)
@@ -1,5 +1,5 @@
 <?xml version="1.0"?>
 <robot xmlns:xacro="http://www.ros.org/wiki/xacro" name="prototype">
-    <xacro:property name="wheel_radius" value="0.0325"/>
+    <xacro:property name="wheel_radius" value="0.032"/>
     <xacro:property name="wheel_length" value="0.026"/>
    <!--===============xacro for continuous joints=========================-->

File: src/prototype/urdf/lidar.xacro (robot description, xacro)
@@ -4,5 +4,5 @@
 <link name="laser_scan_frame">
     <visual>
-        <origin xyz="0 0 0" rpy="0.0 0.0 -1.57"/>
+        <origin xyz="0 0 0" rpy="0.0 0.0 0.0"/>
         <geometry>
            <mesh filename="package://prototype/meshes/sensors/rplidar.dae" scale="1.0 1.0 1.0"/>
@@ -22,5 +22,5 @@
 </link>
 <joint name="laser_scan_frame_joint" type="fixed">
-    <origin xyz="0.0 0.0 0.15" rpy="0.0 0.0 0.0"/>
+    <origin xyz="0.0 0.0 0.15" rpy="0.0 0.0 -1.57"/>
     <!--<parent link="laser_scan_link"/>
     <child link="laser_scan_frame"/>

File: src/prototype/urdf/prototype.xacro (robot description, xacro)
@@ -2,5 +2,4 @@
 <!--=========================starting xacros================================-->
 <robot xmlns:xacro="http://www.ros.org/wiki/xacro" name="prototype">
-<xacro:include filename="$(find gazebo_sim)/urdf/prototype.gazebo.xacro"/>
 <xacro:include filename="$(find prototype)/urdf/wheel.xacro"/>
 <xacro:include filename="$(find prototype)/urdf/lidar.xacro"/>
@@ -40,3 +39,10 @@
  <xacro:box_link name="base_link" mass="1.21" ixx="0.0010803" iyy="0.00010259"
  izz="0.00129793" box="0.155 0.3 0.01"/>-->
+ <joint name="imu_joint" type="fixed">
+  <parent link="chassis"/>
+  <child link="imu_link"/>
+  <origin xyz="0.0 0.0 0.0" rpy="0.0 0.0 0.0"/>
+ </joint>
+ <link name="imu_link">
+ </link>
 </robot>

Commit message: updating the motor_control and proto

File: src/prototype/urdf/hardware_interface.xacro (robot description, xacro)
@@ -7,18 +7,20 @@
     <ros2_control name="PrototypeMotor" type="system">
         <hardware>
-          <plugin>diffdrive_arduino/DiffDriveArduinoHardware</plugin>
-          <!--<plugin>motor_control/MotorControl</plugin>-->
-          <param name="left_wheel_name">front_left_wheel_joint</param>
-          <param name="right_wheel_name">front_right_wheel_joint</param>
+          <!--<plugin>diffdrive_arduino/DiffDriveArduinoHardware</plugin>-->
+          <plugin>motor_control/MotorControl</plugin>
+          <param name="front_left_wheel_name">front_left_wheel_joint</param>
+          <param name="front_right_wheel_name">front_right_wheel_joint</param>
+          <param name="back_left_wheel_name">back_left_wheel_joint</param>
+          <param name="back_right_wheel_name">back_right_wheel_joint</param>
           <param name="loop_rate">30</param>
           <param name="device">/dev/ttyACM0</param>
           <param name="baud_rate">115200</param>
-          <param name="timeout_ms">10000</param>
-          <param name="enc_counts_per_rev">80</param>
+          <param name="timeout">1000</param>
+          <param name="enc_counts_per_rev">120</param>
         </hardware>
         <joint name="front_right_wheel_joint">
           <command_interface name="velocity">
-            <param name="min">-10.0</param>
-            <param name="max">10.0</param>
+            <param name="min">0.0</param>
+            <param name="max">2.0</param>
           </command_interface>
           <state_interface name="position" />
@@ -27,6 +29,22 @@
         <joint name="front_left_wheel_joint">
           <command_interface name="velocity">
-            <param name="min">-10.0</param>
-            <param name="max">10.0</param>
+            <param name="min">0.0</param>
+            <param name="max">2.0</param>
+          </command_interface>
+          <state_interface name="position" />
+          <state_interface name="velocity" />
+        </joint>
+        <joint name="back_right_wheel_joint">
+          <command_interface name="velocity">
+            <param name="min">0.0</param>
+            <param name="max">2.0</param>
+          </command_interface>
+          <state_interface name="position" />
+          <state_interface name="velocity" />
+        </joint>
+        <joint name="back_left_wheel_joint">
+          <command_interface name="velocity">
+            <param name="min">0.0</param>
+            <param name="max">2.0</param>
           </command_interface>
           <state_interface name="position" />

File: src/prototype/urdf/wheel.xacro (robot description, xacro)
@@ -36,5 +36,4 @@
 parent="chassis" child="front_left_wheel" />
 <xacro:wheel wheel_name="front_left_wheel"/>
-<!--
 <xacro:joint name="back_right_wheel_joint" origin="-0.0900 0.12 -0.025"
 parent="chassis" child="back_right_wheel"/>
@@ -42,4 +41,4 @@
 <xacro:joint name="back_left_wheel_joint" origin="0.0900 0.12 -0.025"
 parent="chassis" child="back_left_wheel"/>
-<xacro:wheel  wheel_name="back_left_wheel"/>-->
+<xacro:wheel  wheel_name="back_left_wheel"/>
 </robot>

Commit message: updated the robot model

File: src/prototype/urdf/hardware_interface.xacro (robot description, xacro)
@@ -9,30 +9,12 @@
           <!--<plugin>diffdrive_arduino/DiffDriveArduinoHardware</plugin>-->
           <plugin>motor_control/MotorControl</plugin>
-          <param name="front_left_wheel_name">front_left_wheel_joint</param>
-          <param name="front_right_wheel_name">front_right_wheel_joint</param>
           <param name="back_left_wheel_name">back_left_wheel_joint</param>
           <param name="back_right_wheel_name">back_right_wheel_joint</param>
           <param name="loop_rate">30</param>
-          <param name="device">/dev/serial/by-path/pci-0000:03:00.3-usb-0:2.2:1.0</param>
+          <param name="device">/dev/serial/by-path/pci-0000:03:00.3-usb-0:2:1.0</param>
           <param name="baud_rate">115200</param>
           <param name="timeout">1000</param>
-          <param name="enc_counts_per_rev">120</param>
+          <param name="enc_counts_per_rev">5606</param>
         </hardware>
-        <joint name="front_right_wheel_joint">
-          <command_interface name="velocity">
-            <param name="min">0.0</param>
-            <param name="max">2.0</param>
-          </command_interface>
-          <state_interface name="position" />
-          <state_interface name="velocity" />
-        </joint>
-        <joint name="front_left_wheel_joint">
-          <command_interface name="velocity">
-            <param name="min">0.0</param>
-            <param name="max">2.0</param>
-          </command_interface>
-          <state_interface name="position" />
-          <state_interface name="velocity" />
-        </joint>
         <joint name="back_right_wheel_joint">
           <command_interface name="velocity">

Commit message: adding the updated robot model

File: src/prototype/urdf/hardware_interface.xacro (robot description, xacro)
@@ -9,30 +9,12 @@
           <!--<plugin>diffdrive_arduino/DiffDriveArduinoHardware</plugin>-->
           <plugin>motor_control/MotorControl</plugin>
-          <param name="front_left_wheel_name">front_left_wheel_joint</param>
-          <param name="front_right_wheel_name">front_right_wheel_joint</param>
           <param name="back_left_wheel_name">back_left_wheel_joint</param>
           <param name="back_right_wheel_name">back_right_wheel_joint</param>
           <param name="loop_rate">30</param>
-          <param name="device">/dev/ttyACM0</param>
+          <param name="device">/dev/serial/by-path/pci-0000:03:00.3-usb-0:2:1.0</param>
           <param name="baud_rate">115200</param>
           <param name="timeout">1000</param>
-          <param name="enc_counts_per_rev">120</param>
+          <param name="enc_counts_per_rev">5606</param>
         </hardware>
-        <joint name="front_right_wheel_joint">
-          <command_interface name="velocity">
-            <param name="min">0.0</param>
-            <param name="max">2.0</param>
-          </command_interface>
-          <state_interface name="position" />
-          <state_interface name="velocity" />
-        </joint>
-        <joint name="front_left_wheel_joint">
-          <command_interface name="velocity">
-            <param name="min">0.0</param>
-            <param name="max">2.0</param>
-          </command_interface>
-          <state_interface name="position" />
-          <state_interface name="velocity" />
-        </joint>
         <joint name="back_right_wheel_joint">
           <command_interface name="velocity">
@@ -52,3 +34,31 @@
         </joint>
       </ros2_control>
+<!--
+      <ros2_control name="Imu_Sensor" type="sensor">
+        <hardware>
+          <plugin>imu_interface/Imu_Sensor</plugin>
+          <param name="device">/dev/ttyACM1</param>
+          <param name="baud_rate">115200</param>
+          <param name="timeout_ms">10000</param>
+        </hardware>
+       <sensor name="imu_sensor">
+         <state_interface name="orientation.x"/>
+        <state_interface name="orientation.y"/>
+        <state_interface name="orientation.z"/>
+        <state_interface name="orientation.w"/>
+        <state_interface name="angular_velocity.x"/>
+        <state_interface name="angular_velocity.y"/>
+        <state_interface name="angular_velocity.z"/>
+        <state_interface name="linear_acceleration.x"/>
+        <state_interface name="linear_acceleration.y"/>
+        <state_interface name="linear_acceleration.z"/>
+        <param name="frame_id">imu_link</param>
+        <param name="fx_range">100</param>
+        <param name="fy_range">100</param>
+        <param name="fz_range">100</param>
+        <param name="tx_range">15</param>
+        <param name="ty_range">15</param>
+        <param name="tz_range">15</param>
+       </sensor>
+      </ros2_control>-->
 </robot>

File: src/prototype/urdf/prototype.xacro (robot description, xacro)
@@ -44,5 +44,33 @@
   <origin xyz="0.0 0.0 0.0" rpy="0.0 0.0 0.0"/>
  </joint>
- <link name="imu_link">
+ <link name="imu_link"></link>
+ <joint name="caster_wheel_joint" type="fixed">
+  <parent link="chassis"/>
+  <child link="caster_wheel"/>
+  <axis xyz="0 0 0"/>
+  <origin xyz="0.0 -0.10 -0.020" rpy="0 0 0"/>
+ </joint>
+        <link name="caster_wheel">
+            <visual>
+                <origin xyz="0.0 0.0 0.0" rpy="0.0 0.0 0.0"/>
+                <geometry>
+                 <sphere radius="0.021"/>
+                </geometry>
+                <material name="blue">
+                    <color rgba="0.0 0.0 1.0 1.0"/>
+                </material>
+            </visual>
+            <collision>
+                <origin xyz="0.0 0.0 0.0" rpy="0.0 1.5707 0.0"/>
+                <geometry>
+                    <sphere radius="0.021"/>/>
+                </geometry>
+            </collision>
+            <inertial>
+                <origin rpy="0 0 0" xyz="0 0 0"/>
+                <mass value="0.034"/>
+              <inertia ixx="1.37e-5" ixy="0" ixz="0" iyy="1.37e-5" iyz="0" izz="3.41e-6"/>
+              </inertial>
+              <dynamics damping="0.5" friction="0.1"/>
  </link>
 </robot>

File: src/prototype/urdf/wheel.xacro (robot description, xacro)
@@ -30,10 +30,4 @@
    </xacro:macro>
    <!-- *********************wheel links and joints***************************************-->
- <xacro:joint name="front_right_wheel_joint" origin="-0.0900 -0.12 -0.025"
- parent="chassis" child="front_right_wheel"/>
-<xacro:wheel wheel_name="front_right_wheel"/>
-<xacro:joint name="front_left_wheel_joint" origin="0.0900 -.12 -0.025"
-parent="chassis" child="front_left_wheel" />
-<xacro:wheel wheel_name="front_left_wheel"/>
 <xacro:joint name="back_right_wheel_joint" origin="-0.0900 0.12 -0.025"
 parent="chassis" child="back_right_wheel"/>

Commit message: adding action

File: src/prototype/urdf/hardware_interface.xacro (robot description, xacro)
@@ -5,7 +5,8 @@
 <xacro:include filename="$(find prototype)/urdf/link_macros.xacro"/>
    <!-- ======================ROS2_CONTROL=======================-->
+    <!--
     <ros2_control name="PrototypeMotor" type="system">
-        <hardware>
-          <!--<plugin>diffdrive_arduino/DiffDriveArduinoHardware</plugin>-->
+        <hardware> -->
+          <!--<plugin>diffdrive_arduino/DiffDriveArduinoHardware</plugin>--><!--
           <plugin>motor_control/MotorControl</plugin>
           <param name="back_left_wheel_name">back_left_wheel_joint</param>
@@ -33,5 +34,5 @@
           <state_interface name="velocity" />
         </joint>
-      </ros2_control>
+      </ros2_control> -->
 <!--
       <ros2_control name="Imu_Sensor" type="sensor">

File: src/prototype/urdf/joint_macros.xacro (robot description, xacro)
@@ -5,5 +5,5 @@
    <!--===============xacro for continuous joints=========================-->
     <xacro:macro name="joint_wheel" params="name origin parent child">
-        <joint name="${name}" type="continuous">
+        <joint name="${name}" type="fixed">
             <origin xyz="${origin}" rpy="0.0 0.0 0.0"/>
             <parent link="${parent}"/>

File: src/prototype/urdf/prototype.xacro (robot description, xacro)
@@ -8,4 +8,5 @@
 <xacro:include filename="$(find prototype)/urdf/hardware_interface.xacro"/>
 <xacro:include filename="$(find prototype)/urdf/camera.xacro"/>
+<xacro:include filename="$(find prototype)/urdf/pallet_loader.xacro"/>
 <!--=========================xacro:properties=============================-->
     <xacro:property name="body_length" value="0.41"/>
