Commit message: added nav2 updates

File: src/plane/urdf/plane.xacro (robot description, xacro)
@@ -10,20 +10,17 @@
         <origin xyz="0 0 0.5" rpy="0 0 0" />
         <parent link="world" />
-        <child link="plane" />
+        <child link="imu_link" />
     </joint>
-    <link name="plane">
-    </link>
     <joint name="imu_joint" type="continuous">
-        <origin xyz="0 0 0" rpy="0 0 0" />
-        <parent link="plane" />
+        <origin xyz="0 0 1.0" rpy="0 0 0" />
+        <parent link="world" />
         <child link="imu_link" />
-        <axis xyz="1 0 0"/>
-        <limit effort="100" velocity="1" lower="-1.5708" upper="1.5708" />
+        <axis xyz="0.0 0.0 1.0"/>
     </joint>
     <link name="imu_link">
     <visual>
-      <origin rpy="0 0 1.5708" xyz="0 0 0"/>
+      <origin rpy="0 0 0.0" xyz="0 0 0"/>
       <geometry>
-        <box size="0.5 0.5 0.5"/>
+        <box size="0.05 0.05 0.05"/>
       </geometry>
       <material name="white"/>

File: src/prototype/urdf/prototype.xacro (robot description, xacro)
@@ -21,10 +21,10 @@
     <parent link="base_link"/>
     <child link="base_footprint"/>
-    <origin xyz="0 0 0" rpy="0 0 0"/>
+    <origin xyz="0.0 0.0 0.0" rpy="0 0 0"/>
 </joint>
 <link name="base_footprint">
 </link>
  <joint name="chassis_joint" type="fixed">
-  <origin rpy="0 0 0.0" xyz="0 0 0.062"/>
+  <origin rpy="0.0 0.0 0.0" xyz="0 0 0.062"/>
   <parent link="base_link"/>
   <child link="chassis"/>

Commit message: backup

File: src/plane/urdf/plane.xacro (robot description, xacro)
@@ -10,13 +10,13 @@
         <origin xyz="0 0 0.5" rpy="0 0 0" />
         <parent link="world" />
-        <child link="imu_link" />
+        <child link="plane_link_cam" />
     </joint>
     <joint name="imu_joint" type="continuous">
         <origin xyz="0 0 1.0" rpy="0 0 0" />
         <parent link="world" />
-        <child link="imu_link" />
+        <child link="plane_link_cam" />
         <axis xyz="0.0 0.0 1.0"/>
     </joint>
-    <link name="imu_link">
+    <link name="plane_link_cam">
     <visual>
       <origin rpy="0 0 0.0" xyz="0 0 0"/>

Commit message: updated the ros2 aruco

File: src/plane/urdf/plane.xacro (robot description, xacro)
@@ -12,6 +12,6 @@
         <child link="plane_link_cam" />
     </joint>
-    <joint name="imu_joint" type="continuous">
-        <origin xyz="0 0 1.0" rpy="0 0 0" />
+    <joint name="imu_joint" type="fixed">
+        <origin xyz="1.0 0 1.0" rpy="-1.57 -1.57 0" />
         <parent link="world" />
         <child link="plane_link_cam" />
@@ -20,5 +20,5 @@
     <link name="plane_link_cam">
     <visual>
-      <origin rpy="0 0 0.0" xyz="0 0 0"/>
+      <origin rpy="0.0 0.0 0.0" xyz="0 0 0"/>
       <geometry>
         <box size="0.05 0.05 0.05"/>
